File: hardware/kratos/kratos.kicad_pcb (KiCad board)
At the start: 4 copper layers, 32.3 x 50.5 mm, 21 parts, among them J1 IO Header, J3 Power Terminal, J4 VIN, J5 PJ-102A, U1 AP2138, U2 MIC29300-12, U3 MIC29310-5.0, U4 DS2745U

Commit message: Rev B
Parts:
- removed 12BP: 12V Regulator Bypass, Connector_PinHeader_2.54mm:PinHeader_1x02_P2.54mm_Vertical
- removed C1: 10uF, Capacitor_SMD:C_0805_2012Metric
- removed J5: PJ-102A, digikey-footprints:Barrel_Jack_5.5mmODx2.1mmID_PJ-102A
- removed SW: External Switch, Connector_PinSocket_2.54mm:PinSocket_1x02_P2.54mm_Vertical
- removed U2: MIC29300-12, Package_TO_SOT_SMD:TO-263-3_TabPin2
- C2: value 10uF -> 10uF, 16V
- J3: footprint TerminalBlock:TerminalBlock_bornier-5_P5.08mm -> Connector_PinHeader_2.54mm:PinHeader_1x05_P2.54mm_Vertical
- J4: footprint Connector_JST:JST_EH_B02B-EH-A_1x02_P2.50mm_Vertical -> Connector_PinHeader_2.54mm:PinHeader_1x02_P2.54mm_Vertical
- R1: value 15m -> 10m
- R3: value 42k -> 20k
- R5: value 10k -> 4.7k
- moved C3 57.3 mm to (149.1, 114.6), turned to 90 degrees
- moved R2 54.9 mm to (146.8, 114.6), turned to 270 degrees
- moved R1 49.8 mm to (137.2, 99.3)
- moved J3 44.3 mm to (140.0, 88.4), turned to 90 degrees
- moved D1 43.2 mm to (132.3, 88.4)
- moved R6 43.2 mm to (132.3, 90.7)
- moved J1 43.1 mm to (132.0, 96.5)
- moved U1 40.4 mm to (147.1, 92.5), turned to 0 degrees
- moved U4 39.9 mm to (137.2, 108.2), turned to 270 degrees
- moved R3 39.5 mm to (144.5, 114.6), turned to 270 degrees
- moved VBAT1 39.3 mm to (137.2, 114.6)
- moved C2 37.2 mm to (151.4, 114.6), turned to 270 degrees
- moved R4 37.0 mm to (142.2, 114.6), turned to 90 degrees
- moved R5 35.4 mm to (140.0, 114.6), turned to 90 degrees
- moved J4 34.6 mm to (132.1, 113.0), turned to 180 degrees
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Connections:
- J3 pad 2: +12V -> +5V
- J3 pad 3: +5V -> Net-(J3-Pad3)
- J4 pad 1: Net-(J4-Pad1) -> VDC
- U3 pad 1: +12V -> VDC
Routing:
- net /Input/rsense+: track 25.3 -> 6.40 mm, vias 2 -> 3
- net GND: track 20.6 -> 3.43 mm, vias 96 -> 23
- net +3V3: track 53.2 -> 37.4 mm, vias 2 -> 0
- net /p1: track 18.1 -> 9.23 mm
- net Net-(R3-Pad2): track 15.8 -> 7.74 mm
- net /sda: track 20.2 -> 12.1 mm
- net +12V: track 7.47 -> 0.00 mm, vias 6 -> 0
- net +5V: track 24.3 -> 16.9 mm
- net /scl: track 21.6 -> 15.0 mm
- net Net-(C3-Pad2): track 11.0 -> 14.1 mm, vias 2 -> 0
- net Net-(R4-Pad2): track 6.29 -> 7.84 mm
- net Net-(C3-Pad1): track 3.30 -> 2.30 mm
- net VDC: track 2.91 -> 2.29 mm, vias 5 -> 4
- added copper zone on F.Cu, net (none)
- removed copper zone on PWR, net +12V
- removed copper zone on B.Cu, net GND
- removed copper zone on F.Cu, net GND
- removed copper zone on PWR, net Net-(J4-Pad1)
Other:
- board size 32.3 x 50.5 mm -> 23.1 x 32.8 mm
- board text added: "+ 5 N 3 G"
- board text added: "kratos-pdb :: Rev B nnarain"
- board text removed: "12V"
- board text removed: "3V3"
- board text removed: "5V"
- board text removed: "GND"
- board text removed: "P1"
- board text removed: "PWR"
- board text removed: "RAW"
- board text removed: "SCL"
- board text removed: "SDA"
- board text removed: "kratos"
- board text removed: "kratos-pdb :: REVA nnarain"
