File: hardware/kratos/kratos.kicad_sch (KiCad schematic)
At the start: 27 parts, among them J1 BATT, J10 PWM4, J11 PWM5, J12 PWM6, J6 VCC_SEL, J7 PWM1, J8 PWM2, J9 PWM3, U1 TPS5430DDA, U2 AMS1117-3.3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

Commit message: Fix 10k resistor JLCPCB selection
Parts:
- R1, R2: LCSC C17408 -> C17414
Changed lines of the file:
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@@
       (effects (font (size 1.27 1.27)) hide)
     )
-    (property "LCSC" "C17408" (id 4) (at 179.07 33.02 0)
+    (property "LCSC" "C17414" (id 4) (at 179.07 33.02 0)
       (effects (font (size 1.27 1.27)) hide)
     )
@@
       (effects (font (size 1.27 1.27)) hide)
     )
-    (property "LCSC" "C17408" (id 4) (at 90.17 38.1 90)
+    (property "LCSC" "C17414" (id 4) (at 90.17 38.1 90)
       (effects (font (size 1.27 1.27)) hide)
     )
